Commit message: Created a runable script to place in workspace that launches bringup made robot show in world and updated bringup (still needs changes for teleop) also fixed mistakes in robot description

File: robutler_description/urdf/robutler.gazebo.xacro (robot description, xacro)
@@ -6,5 +6,5 @@
   <gazebo reference="base_link">
     <!-- <material>Gazebo/DarkGrey</material> -->
-    <material>Gazebo/Turquoise</material>
+    <material>Gazebo/Blue</material>
   </gazebo>
   <gazebo reference="wheel_left_link">
@@ -17,5 +17,5 @@
     <fdir1>1 0 0</fdir1>
     <!-- <material>Gazebo/FlatBlack</material> -->
-    <material>Gazebo/Yellow</material>
+    <material>Gazebo/Red</material>
   </gazebo>
   <gazebo reference="wheel_right_link">
@@ -28,5 +28,5 @@
     <fdir1>1 0 0</fdir1>
     <!-- <material>Gazebo/FlatBlack</material> -->
-    <material>Gazebo/Yellow</material>
+    <material>Gazebo/Red</material>
   </gazebo>
   <gazebo reference="caster_back_right_link">
@@ -111,5 +111,4 @@
       <pose>0 0 0 0 0 0</pose>
       <visualize>$(arg laser_visual)</visualize>
-      <!-- <visualize>true</visualize> -->
       <update_rate>5</update_rate>
       <ray>

File: robutler_description/urdf/robutler.urdf.xacro (robot description, xacro)
@@ -16,5 +16,5 @@
       </geometry>
       <!-- <material name="light_black"/> -->
-      <material name="turquoise"/>
+      <material name="blue"/>
     </visual>
     <collision>
@@ -44,5 +44,5 @@
         <mesh filename="package://turtlebot3_description/meshes/wheels/left_tire.stl" scale="0.001 0.001 0.001"/>
       </geometry>
-      <material name="blue"/>
+      <material name="red"/>
     </visual>
     <collision>
@@ -72,5 +72,5 @@
         <mesh filename="package://turtlebot3_description/meshes/wheels/right_tire.stl" scale="0.001 0.001 0.001"/>
       </geometry>
-      <material name="blue"/>
+      <material name="red"/>
     </visual>
     <collision>
@@ -145,5 +145,5 @@
         <mesh filename="package://turtlebot3_description/meshes/sensors/lds.stl" scale="0.001 0.001 0.001"/>
       </geometry>
-      <material name="blue"/>
+      <material name="dark"/>
     </visual>
     <collision>
@@ -161,8 +161,23 @@
     </inertial>
   </link>
+  <!-- Connect Camera to the base -->
+  <link name="camera_to_base">
+    <visual>
+      <geometry>
+        <cylinder length="1" radius="0.02"/>
+      </geometry>
+      <material name="blue"/>
+    </visual>
+  </link>
+  <joint name="camera_to_base_joint" type="fixed">
+    <!-- <origin xyz="0.073 -0.011 0.084" rpy="0 0 0"/> -->
+    <origin xyz="0.033 0 0.5" rpy="0 0 0"/>
+    <parent link="base_link"/>
+    <child link="camera_to_base"/>
+  </joint>
   <joint name="camera_joint" type="fixed">
     <!-- <origin xyz="0.073 -0.011 0.084" rpy="0 0 0"/> -->
-    <origin xyz="0.073 -0.011 1" rpy="0 0 0"/>
-    <parent link="base_link"/>
+    <origin xyz="0 0 0.5" rpy="0 0 0"/>
+    <parent link="camera_to_base"/>
     <child link="camera_link"/>
   </joint>
