Commit message: Read me is now decent

File: robutler_description/urdf/robutler.urdf.xacro (robot description, xacro)
@@ -171,11 +171,9 @@
   </link>
   <joint name="camera_to_base_joint" type="fixed">
-    <!-- <origin xyz="0.073 -0.011 0.084" rpy="0 0 0"/> -->
-    <origin xyz="0.033 0 0.5" rpy="0 0 0"/>
+    <origin xyz="0.073 -0.011 0.5" rpy="0 0 0"/>
     <parent link="base_link"/>
     <child link="camera_to_base"/>
   </joint>
   <joint name="camera_joint" type="fixed">
-    <!-- <origin xyz="0.073 -0.011 0.084" rpy="0 0 0"/> -->
     <origin xyz="0 0 0.5" rpy="0 0 0"/>
     <parent link="camera_to_base"/>
